File: drv8301.kicad_sch (KiCad schematic)
At the start: 48 parts, among them Q1 DMN62D0UW, U2 Mc74VHC1GT66, U3 DRV8301DCAR, U4 Mc74VHC1GT66, U5 Mc74VHC1GT66, U6 TLV73333PDBV

Commit message: Update
Parts:
- removed C16: 2.2u, Capacitor_SMD:C_0805_2012Metric, symbol Device:C
- added C1, C2: 100n, Capacitor_SMD:C_0603_1608Metric, symbol Device:C
- C17, C18, C21: footprint Capacitor_SMD:C_0805_2012Metric -> Capacitor_SMD:C_0603_1608Metric_Pad1.08x0.95mm_HandSolder; Voltage 100V -> 25V
- C20, C23, C26, C27, C35, C36: Voltage 50V -> 100V
- C28, C29, C30: Voltage 100V -> 25V
Connections:
- net GND: now also C1.2, C2.2
- net SUPPLY: no longer R28.1
- net Supply_Filterted: now also R28.1, C1.1, C2.1
- net at C22.1, U3.14 (CP1): no longer C17.1, U3.13 (GVDD)
- new net: C17.1, U3.13 (GVDD)
Other:
- moved on the sheet: C17, C22, C25, C31, C32, C56, C58, FB1, R20, R21, R24, R25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
