File: power.kicad_sch (KiCad schematic)
At the start: 44 parts, among them Q2 HYG015N10NS1TA, Q3 HYG015N10NS1TA, Q4 HYG015N10NS1TA, Q5 HYG015N10NS1TA, Q6 HYG015N10NS1TA, Q7 HYG015N10NS1TA, U10 AD8418, U11 Mc74VHC1GT66, U12 AD8418, U7 AD8418, U8 Mc74VHC1GT66, U9 Mc74VHC1GT66

Commit message: Update
Parts:
- removed R31, R35, R39: 0.5m, TUWR_Sensors:BVN_1216, symbol Device:R_Shunt
- added C16, C68, C76: 1n, Capacitor_SMD:C_0603_1608Metric, symbol Device:C
- added R49, R53, R57: 0.5m, TUWR_Sensors:WSLP3921, symbol Device:R
- C59: renamed from C38; Voltage 50V -> 100V
- C67: renamed from C43; footprint Capacitor_THT:CP_Radial_D12.5mm_P5.00mm -> Capacitor_THT:CP_Radial_D10.0mm_P5.00mm
- C69: renamed from C44; Voltage 50V -> 100V
- C70: renamed from C45; footprint Capacitor_THT:CP_Radial_D12.5mm_P5.00mm -> Capacitor_THT:CP_Radial_D10.0mm_P5.00mm
- C72: renamed from C47; footprint Capacitor_THT:CP_Radial_D12.5mm_P5.00mm -> Capacitor_THT:CP_Radial_D10.0mm_P5.00mm
- C77: renamed from C51; Voltage 50V -> 100V
- renumbered C39 to C60, C40 to C64, C41 to C65, C42 to C66, C46 to C71, C48 to C73, C49 to C74, C50 to C75, C52 to C78, C53 to C79, C54 to C80, C55 to C81, Q4 to Q10, Q5 to Q11, Q6 to Q12, Q7 to Q13, Q2 to Q8, Q3 to Q9, R30 to R48, R32 to R50, R33 to R51, R34 to R52, R36 to R54, R37 to R55, R38 to R56, R40 to R58, R41 to R59, R42 to R60, TH1 to TH2, U7 to U13, U8 to U15, U9 to U16, U10 to U17, U11 to U18, U12 to U19
Connections:
- net SH_A is gone; now on net SH_A_P: Q8.2 (S), Q9.3 (D)
- net SH_B is gone; now on net SH_B_P: Q10.2 (S), Q11.3 (D)
- net SH_C is gone; now on net SH_C_P: Q12.2 (S), Q13.3 (D)
- net SH_B_P: now reaches U17.1 (IN-)
- net SH_B_P: now also C68.1, R53.1
- net SH_B_N: now reaches U17.8 (IN+)
- net SH_B_N: now also C68.2, R53.2
- net SH_C_N: now reaches U19.8 (IN+)
- net SH_C_N: now also C76.2, R49.2
- net SH_C_P: now reaches U19.1 (IN-)
- net SH_C_P: now also C76.1, R49.1
- net SH_A_N: now reaches U13.8 (IN+)
- net SH_A_N: now also C16.2, R57.2
- net SH_A_P: now reaches U13.1 (IN-)
- net SH_A_P: now also C16.1, R57.1
Other:
- moved on the sheet: C59, C60, C64, C65, C66, C67, C69, C73, C74, C75, C77, C78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
