File: vesc6.kicad_sch (KiCad schematic)
At the start: 1 part, among them J1 Main

Commit message: Update
Parts:
- added H1: MountingHole_Pad, MountingHole:MountingHole_3.7mm_Pad_Via, symbol Mechanical:MountingHole_Pad
Connections:
- net GND: now also H1.1
- net VESC_Right/CAN_H renamed VESC_Left/CAN_H
- net VESC_Right/CAN_L renamed VESC_Left/CAN_L
Other:
- added sheet VESC_Left (vesc_left.kicad_sch)
- sheet VESC_Right: file vesc_left.kicad_sch -> vesc_right.kicad_sch
- sheet VESC_Right ports: added SUPPLY; removed none
